File: BSPD-Logic.kicad_sch (KiCad schematic)
At the start: 84 parts, among them IC1 MCP1804T-C002I/OT, Q11 SI2347DS-T1-GE3, Q12 SI2347DS-T1-GE3, Q14 MMBT3904L RFG, Q17 MMBT3904L RFG, U1 LM393BIDR, U2 LM393BIDR, U4 LM393BIDR, U5 CD4002BM96, U6 LM393BIDR

Commit message: completed schematic cleanup, back on 12V
Parts:
- renumbered C5 to C10, C4 to C11, C3 to C4, C8 to C5, C11 to C6, C6 to C8, C2 to C9, D40 to D12, D11 to D13, D39 to D14, D41 to D15, D14 to D16, D38 to D17, Q14 to Q10, Q17 to Q11, Q11 to Q8, Q12 to Q9, R58 to R19, R59 to R20, R87 to R21, R88 to R22, R36 to R23, R86 to R24, R92 to R25, R90 to R26, R89 to R27, R91 to R28, R80 to R29, R81 to R30, R82 to R31, R83 to R32, R28 to R33, R10 to R34, R43 to R35, R31 to R36, R54 to R37, R53 to R38, R45 to R39, R44 to R40, R29 to R41, R24 to R42, R56 to R43, R62 to R44, R61 to R45, R77 to R46, R55 to R47, R49 to R48, R72 to R49, R76 to R50, R46 to R51, R50 to R52, R52 to R53, R71 to R54, RV4 to RV2, RV5 to RV3, RV6 to RV4, RV2 to RV5, RV3 to RV6, TP15 to TP10, TP10 to TP11, TP11 to TP12, TP17 to TP13, TP20 to TP14, TP21 to TP15, TP22 to TP16, TP23 to TP17, TP24 to TP18, TP16 to TP19, TP13 to TP20, TP18 to TP21, TP19 to TP22, TP27 to TP23, TP26 to TP6, TP9 to TP7, TP12 to TP8, TP14 to TP9, U6 to U1, U1 to U2, U4 to U3, U2 to U3, U6 to U4
Connections:
- net GND: now also U1.5 (+)
- net at U1.6 (-): now also U1.7
- net ACCUM-VOUT renamed ISENSE-EXT
- net BRAKE-VOUT renamed BSE
- no-connect marks 6 -> 3
Other:
- moved on the sheet: Q10, Q11, R51, R52, TP22, TP23, U1B

Commit message: completed placement:
Parts:
- removed TP13, TP14, TP15, TP16, TP17, TP18: ~, TestPoint:TestPoint_Pad_1.5x1.5mm, symbol -Test-Points:Square-Pad-1.5mm
- U3: renamed from IC1; footprint -LDO:SOT95P270X145-5N -> Package_TO_SOT_SMD:SOT-23-5
- renumbered C7 to C4, C8 to C5, C4 to C6, C5 to C7, C6 to C8, D15 to D12, D16 to D13, D17 to D14, D12 to D15, D13 to D16, D14 to D17, Q8 to Q10, Q9 to Q8, Q10 to Q9, R21 to R19, R22 to R20, R19 to R21, R27 to R22, R44 to R23, R23 to R24, R37 to R25, R45 to R26, R47 to R27, R50 to R28, R43 to R29, R20 to R30, R53 to R31, R54 to R32, R24 to R33, R38 to R34, R28 to R35, R25 to R36, R26 to R37, R29 to R38, R51 to R39, R39 to R40, R35 to R41, R48 to R42, R49 to R43, R33 to R44, R52 to R45, R40 to R46, R46 to R47, R30 to R48, R31 to R49, R41 to R50, R36 to R51, R34 to R52, R42 to R53, R32 to R54, TP22 to TP10, TP8 to TP11, TP19 to TP13, TP23 to TP14, TP9 to TP15, TP10 to TP17, TP21 to TP19, TP11 to TP20, TP12 to TP22, TP7 to TP6, TP20 to TP8, TP6 to TP9, U2 to U1, U4 to U2, U1 to U2, U5 to U4, U3 to U5, U2 to U5, U4 to U6, U3 to U6
