File: Fault-Passthru.kicad_sch (KiCad schematic)
At the start: 12 parts, among them Q10 SI2318CDS-T1-GE3, Q7 SI2347DS-T1-GE3

Commit message: completed schematic cleanup, back on 12V
Parts:
- renumbered D13 to D18, D16 to D19, D15 to D20, D37 to D21, Q7 to Q12, Q10 to Q13, R8 to R55, R15 to R56, R27 to R57, R30 to R58, R75 to R59, R70 to R60
Connections:
- net ERROR-OUT renamed ERROR-SIG

Commit message: completed placement:
Parts:
- renumbered D21 to D20, D20 to D21, R58 to R55, R60 to R56, R55 to R57, R56 to R58, R57 to R59, R59 to R60
Changed lines of the file:
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@@
 		(on_board yes)
 		(dnp no)
-		(property "Reference" "R56"
+		(property "Reference" "R58"
 			(at 184.7056 147.6295 90)
 			(effects
@@
 			(project "Shutdown"
 				(path "/624b8e71-6fec-49ba-b7c9-b659e140fc2f/2f9ac893-2047-438f-af87-5654fc0cb14f"
-					(reference "R56")
+					(reference "R58")
 					(unit 1)
 				)
 				(path "/624b8e71-6fec-49ba-b7c9-b659e140fc2f/5fbdbc4a-acfc-4802-ab24-0d194c32f3aa"
-					(reference "R68")
+					(reference "R70")
 					(unit 1)
 				)
 				(path "/624b8e71-6fec-49ba-b7c9-b659e140fc2f/6ab0f091-adec-4d1f-a1d7-0124abb21b07"
-					(reference "R62")
+					(reference "R64")
 					(unit 1)
 				)
@@
 		(on_board yes)
 		(dnp no)
-		(property "Reference" "R59"
+		(property "Reference" "R60"
 			(at 222.8921 170.8631 90)
 			(effects
@@
 			(project "Shutdown"
 				(path "/624b8e71-6fec-49ba-b7c9-b659e140fc2f/2f9ac893-2047-438f-af87-5654fc0cb14f"
-					(reference "R59")
+					(reference "R60")
 					(unit 1)
 				)
 				(path "/624b8e71-6fec-49ba-b7c9-b659e140fc2f/5fbdbc4a-acfc-4802-ab24-0d194c32f3aa"
-					(reference "R71")
+					(reference "R72")
 					(unit 1)
 				)
 				(path "/624b8e71-6fec-49ba-b7c9-b659e140fc2f/6ab0f091-adec-4d1f-a1d7-0124abb21b07"
-					(reference "R65")
+					(reference "R66")
 					(unit 1)
 				)
@@
 		(on_board yes)
 		(dnp no)
-		(property "Reference" "D21"
+		(property "Reference" "D20"
 			(at 235.5885 145.2833 90)
 			(effects
@@
 			(project "Shutdown"
 				(path "/624b8e71-6fec-49ba-b7c9-b659e140fc2f/2f9ac893-2047-438f-af87-5654fc0cb14f"
-					(reference "D21")
+					(reference "D20")
 					(unit 1)
 				)
 				(path "/624b8e71-6fec-49ba-b7c9-b659e140fc2f/5fbdbc4a-acfc-4802-ab24-0d194c32f3aa"
-					(reference "D29")
+					(reference "D28")
 					(unit 1)
 				)
 				(path "/624b8e71-6fec-49ba-b7c9-b659e140fc2f/6ab0f091-adec-4d1f-a1d7-0124abb21b07"
-					(reference "D25")
+					(reference "D24")
 					(unit 1)
 				)
@@
 		(on_board yes)
 		(dnp no)
-		(property "Reference" "#PWR078"
+		(property "Reference" "#PWR077"
 			(at 220.98 189.23 0)
 			(effects
@@
 			(project "Shutdown"
 				(path "/624b8e71-6fec-49ba-b7c9-b659e140fc2f/2f9ac893-2047-438f-af87-5654fc0cb14f"
-					(reference "#PWR078")
+					(reference "#PWR077")
 					(unit 1)
 				)
 				(path "/624b8e71-6fec-49ba-b7c9-b659e140fc2f/5fbdbc4a-acfc-4802-ab24-0d194c32f3aa"
-					(reference "#PWR084")
+					(reference "#PWR083")
 					(unit 1)
 				)
 				(path "/624b8e71-6fec-49ba-b7c9-b659e140fc2f/6ab0f091-adec-4d1f-a1d7-0124abb21b07"
-					(reference "#PWR081")
+					(reference "#PWR080")
 					(unit 1)
 				)
@@
 		(on_board yes)
 		(dnp no)
-		(property "Reference" "R58"
+		(property "Reference" "R55"
 			(at 222.588 131.7328 90)
 			(effects
@@
 			(project "Shutdown"
 				(path "/624b8e71-6fec-49ba-b7c9-b659e140fc2f/2f9ac893-2047-438f-af87-5654fc0cb14f"
-					(reference "R58")
+					(reference "R55")
 					(unit 1)
 				)
 				(path "/624b8e71-6fec-49ba-b7c9-b659e140fc2f/5fbdbc4a-acfc-4802-ab24-0d194c32f3aa"
-					(reference "R70")
+					(reference "R67")
 					(unit 1)
 				)
 				(path "/624b8e71-6fec-49ba-b7c9-b659e140fc2f/6ab0f091-adec-4d1f-a1d7-0124abb21b07"
-					(reference "R64")
+					(reference "R61")
 					(unit 1)
 				)
@@
 		(on_board yes)
 		(dnp no)
-		(property "Reference" "R57"
+		(property "Reference" "R59"
 			(at 201.804 162.8047 0)
 			(effects
@@
 			(project "Shutdown"
 				(path "/624b8e71-6fec-49ba-b7c9-b659e140fc2f/2f9ac893-2047-438f-af87-5654fc0cb14f"
-					(reference "R57")
+					(reference "R59")
 					(unit 1)
 				)
 				(path "/624b8e71-6fec-49ba-b7c9-b659e140fc2f/5fbdbc4a-acfc-4802-ab24-0d194c32f3aa"
-					(reference "R69")
+					(reference "R71")
 					(unit 1)
 				)
 				(path "/624b8e71-6fec-49ba-b7c9-b659e140fc2f/6ab0f091-adec-4d1f-a1d7-0124abb21b07"
-					(reference "R63")
+					(reference "R65")
 					(unit 1)
 				)
@@
 		(on_board yes)
 		(dnp no)
-		(property "Reference" "R60"
+		(property "Reference" "R56"
 			(at 234.018 131.7328 90)
 			(effects
@@
 			(project "Shutdown"
 				(path "/624b8e71-6fec-49ba-b7c9-b659e140fc2f/2f9ac893-2047-438f-af87-5654fc0cb14f"
-					(reference "R60")
+					(reference "R56")
 					(unit 1)
 				)
 				(path "/624b8e71-6fec-49ba-b7c9-b659e140fc2f/5fbdbc4a-acfc-4802-ab24-0d194c32f3aa"
-					(reference "R72")
+					(reference "R68")
 					(unit 1)
 				)
 				(path "/624b8e71-6fec-49ba-b7c9-b659e140fc2f/6ab0f091-adec-4d1f-a1d7-0124abb21b07"
-					(reference "R66")
+					(reference "R62")
 					(unit 1)
 				)
@@
 		(on_board yes)
 		(dnp no)
-		(property "Reference" "R55"
+		(property "Reference" "R57"
 			(at 169.4656 147.6295 90)
 			(effects
@@
 			(project "Shutdown"
 				(path "/624b8e71-6fec-49ba-b7c9-b659e140fc2f/2f9ac893-2047-438f-af87-5654fc0cb14f"
-					(reference "R55")
+					(reference "R57")
 					(unit 1)
 				)
 				(path "/624b8e71-6fec-49ba-b7c9-b659e140fc2f/5fbdbc4a-acfc-4802-ab24-0d194c32f3aa"
-					(reference "R67")
+					(reference "R69")
 					(unit 1)
 				)
 				(path "/624b8e71-6fec-49ba-b7c9-b659e140fc2f/6ab0f091-adec-4d1f-a1d7-0124abb21b07"
-					(reference "R61")
+					(reference "R63")
 					(unit 1)
 				)
@@
 		(on_board yes)
 		(dnp no)
-		(property "Reference" "D20"
+		(property "Reference" "D21"
 			(at 213.0765 169.2859 0)
 			(effects
@@
 			(project "Shutdown"
 				(path "/624b8e71-6fec-49ba-b7c9-b659e140fc2f/2f9ac893-2047-438f-af87-5654fc0cb14f"
-					(reference "D20")
+					(reference "D21")
 					(unit 1)
 				)
 				(path "/624b8e71-6fec-49ba-b7c9-b659e140fc2f/5fbdbc4a-acfc-4802-ab24-0d194c32f3aa"
-					(reference "D28")
+					(reference "D29")
 					(unit 1)
 				)
 				(path "/624b8e71-6fec-49ba-b7c9-b659e140fc2f/6ab0f091-adec-4d1f-a1d7-0124abb21b07"
-					(reference "D24")
+					(reference "D25")
 					(unit 1)
 				)
@@
 		(on_board yes)
 		(dnp no)
-		(property "Reference" "#PWR077"
+		(property "Reference" "#PWR075"
 			(at 220.98 129.54 0)
 			(effects
@@
 			(project "Shutdown"
 				(path "/624b8e71-6fec-49ba-b7c9-b659e140fc2f/2f9ac893-2047-438f-af87-5654fc0cb14f"
-					(reference "#PWR077")
+					(reference "#PWR075")
 					(unit 1)
 				)
 				(path "/624b8e71-6fec-49ba-b7c9-b659e140fc2f/5fbdbc4a-acfc-4802-ab24-0d194c32f3aa"
-					(reference "#PWR083")
+					(reference "#PWR081")
 					(unit 1)
 				)
 				(path "/624b8e71-6fec-49ba-b7c9-b659e140fc2f/6ab0f091-adec-4d1f-a1d7-0124abb21b07"
-					(reference "#PWR080")
-					(unit 1)
-				)
+					(reference "#PWR078")
+					(unit 1)
+				)
