File: Fault-Passthru.kicad_sch (KiCad schematic)
At the start: 12 parts, among them Q12 SI2347DS-T1-GE3, Q13 SI2318CDS-T1-GE3

Commit message: updated port directionalities, updated pinout
Changed lines of the file:
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@@
 	)
 	(hierarchical_label "OUTPUT"
-		(shape input)
+		(shape output)
 		(at 201.93 133.35 0)
 		(effects

Commit message: Schem is reannotated time to redo all of the layout
Parts:
- renumbered D18 to D16, D19 to D17, D20 to D18, D21 to D19, R55 to R32, R56 to R33, R57 to R34, R58 to R35, R59 to R36, R60 to R37
Changed lines of the file:
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@@
 		(on_board yes)
 		(dnp no)
-		(property "Reference" "R58"
+		(property "Reference" "R35"
 			(at 184.7056 147.6295 90)
 			(effects
@@
 			(project "Shutdown"
 				(path "/624b8e71-6fec-49ba-b7c9-b659e140fc2f/2f9ac893-2047-438f-af87-5654fc0cb14f"
-					(reference "R58")
+					(reference "R35")
 					(unit 1)
 				)
 				(path "/624b8e71-6fec-49ba-b7c9-b659e140fc2f/5fbdbc4a-acfc-4802-ab24-0d194c32f3aa"
-					(reference "R70")
+					(reference "R41")
 					(unit 1)
 				)
@@
 		(on_board yes)
 		(dnp no)
-		(property "Reference" "R60"
+		(property "Reference" "R37"
 			(at 222.8921 170.8631 90)
 			(effects
@@
 			(project "Shutdown"
 				(path "/624b8e71-6fec-49ba-b7c9-b659e140fc2f/2f9ac893-2047-438f-af87-5654fc0cb14f"
-					(reference "R60")
+					(reference "R37")
 					(unit 1)
 				)
 				(path "/624b8e71-6fec-49ba-b7c9-b659e140fc2f/5fbdbc4a-acfc-4802-ab24-0d194c32f3aa"
-					(reference "R72")
+					(reference "R43")
 					(unit 1)
 				)
@@
 		(on_board yes)
 		(dnp no)
-		(property "Reference" "D20"
+		(property "Reference" "D18"
 			(at 235.5885 145.2833 90)
 			(effects
@@
 			(project "Shutdown"
 				(path "/624b8e71-6fec-49ba-b7c9-b659e140fc2f/2f9ac893-2047-438f-af87-5654fc0cb14f"
-					(reference "D20")
+					(reference "D18")
 					(unit 1)
 				)
 				(path "/624b8e71-6fec-49ba-b7c9-b659e140fc2f/5fbdbc4a-acfc-4802-ab24-0d194c32f3aa"
-					(reference "D28")
+					(reference "D22")
 					(unit 1)
 				)
@@
 				)
 				(path "/624b8e71-6fec-49ba-b7c9-b659e140fc2f/5fbdbc4a-acfc-4802-ab24-0d194c32f3aa"
-					(reference "Q17")
+					(reference "Q15")
 					(unit 1)
 				)
@@
 		(on_board yes)
 		(dnp no)
-		(property "Reference" "#PWR077"
+		(property "Reference" "#PWR039"
 			(at 220.98 189.23 0)
 			(effects
@@
 			(project "Shutdown"
 				(path "/624b8e71-6fec-49ba-b7c9-b659e140fc2f/2f9ac893-2047-438f-af87-5654fc0cb14f"
-					(reference "#PWR077")
+					(reference "#PWR039")
 					(unit 1)
 				)
 				(path "/624b8e71-6fec-49ba-b7c9-b659e140fc2f/5fbdbc4a-acfc-4802-ab24-0d194c32f3aa"
-					(reference "#PWR083")
+					(reference "#PWR042")
 					(unit 1)
 				)
@@
 		(on_board yes)
 		(dnp no)
-		(property "Reference" "R55"
+		(property "Reference" "R32"
 			(at 222.588 131.7328 90)
 			(effects
@@
 			(project "Shutdown"
 				(path "/624b8e71-6fec-49ba-b7c9-b659e140fc2f/2f9ac893-2047-438f-af87-5654fc0cb14f"
-					(reference "R55")
+					(reference "R32")
 					(unit 1)
 				)
 				(path "/624b8e71-6fec-49ba-b7c9-b659e140fc2f/5fbdbc4a-acfc-4802-ab24-0d194c32f3aa"
-					(reference "R67")
+					(reference "R38")
 					(unit 1)
 				)
@@
 		(on_board yes)
 		(dnp no)
-		(property "Reference" "R59"
+		(property "Reference" "R36"
 			(at 201.804 162.8047 0)
 			(effects
@@
 			(project "Shutdown"
 				(path "/624b8e71-6fec-49ba-b7c9-b659e140fc2f/2f9ac893-2047-438f-af87-5654fc0cb14f"
-					(reference "R59")
+					(reference "R36")
 					(unit 1)
 				)
 				(path "/624b8e71-6fec-49ba-b7c9-b659e140fc2f/5fbdbc4a-acfc-4802-ab24-0d194c32f3aa"
-					(reference "R71")
+					(reference "R42")
 					(unit 1)
 				)
@@
 		(on_board yes)
 		(dnp no)
-		(property "Reference" "R56"
+		(property "Reference" "R33"
 			(at 234.018 131.7328 90)
 			(effects
@@
 			(project "Shutdown"
 				(path "/624b8e71-6fec-49ba-b7c9-b659e140fc2f/2f9ac893-2047-438f-af87-5654fc0cb14f"
-					(reference "R56")
+					(reference "R33")
 					(unit 1)
 				)
 				(path "/624b8e71-6fec-49ba-b7c9-b659e140fc2f/5fbdbc4a-acfc-4802-ab24-0d194c32f3aa"
-					(reference "R68")
+					(reference "R39")
 					(unit 1)
 				)
@@
 		(on_board yes)
 		(dnp no)
-		(property "Reference" "R57"
+		(property "Reference" "R34"
 			(at 169.4656 147.6295 90)
 			(effects
@@
 			(project "Shutdown"
 				(path "/624b8e71-6fec-49ba-b7c9-b659e140fc2f/2f9ac893-2047-438f-af87-5654fc0cb14f"
-					(reference "R57")
+					(reference "R34")
 					(unit 1)
 				)
 				(path "/624b8e71-6fec-49ba-b7c9-b659e140fc2f/5fbdbc4a-acfc-4802-ab24-0d194c32f3aa"
-					(reference "R69")
+					(reference "R40")
 					(unit 1)
 				)
@@
 		(on_board yes)
 		(dnp no)
-		(property "Reference" "D18"
+		(property "Reference" "D16"
 			(at 182.784 128.0941 90)
 			(effects
@@
 			(project "Shutdown"
 				(path "/624b8e71-6fec-49ba-b7c9-b659e140fc2f/2f9ac893-2047-438f-af87-5654fc0cb14f"
-					(reference "D18")
+					(reference "D16")
 					(unit 1)
 				)
 				(path "/624b8e71-6fec-49ba-b7c9-b659e140fc2f/5fbdbc4a-acfc-4802-ab24-0d194c32f3aa"
-					(reference "D26")
+					(reference "D20")
 					(unit 1)
 				)
@@
 		(on_board yes)
 		(dnp no)
-		(property "Reference" "D21"
+		(property "Reference" "D19"
 			(at 213.0765 169.2859 0)
 			(effects
@@
 			(project "Shutdown"
 				(path "/624b8e71-6fec-49ba-b7c9-b659e140fc2f/2f9ac893-2047-438f-af87-5654fc0cb14f"
-					(reference "D21")
+					(reference "D19")
 					(unit 1)
 				)
 				(path "/624b8e71-6fec-49ba-b7c9-b659e140fc2f/5fbdbc4a-acfc-4802-ab24-0d194c32f3aa"
-					(reference "D29")
+					(reference "D23")
 					(unit 1)
 				)
@@
 		(on_board yes)
 		(dnp no)
-		(property "Reference" "D19"
+		(property "Reference" "D17"
 			(at 224.1585 145.2833 90)
 			(effects
@@
 			(project "Shutdown"
 				(path "/624b8e71-6fec-49ba-b7c9-b659e140fc2f/2f9ac893-2047-438f-af87-5654fc0cb14f"
-					(reference "D19")
+					(reference "D17")
 					(unit 1)
 				)
 				(path "/624b8e71-6fec-49ba-b7c9-b659e140fc2f/5fbdbc4a-acfc-4802-ab24-0d194c32f3aa"
-					(reference "D27")
+					(reference "D21")
 					(unit 1)
 				)
@@
 		(on_board yes)
 		(dnp no)
-		(property "Reference" "#PWR075"
+		(property "Reference" "#PWR037"
 			(at 220.98 129.54 0)
 			(effects
@@
 			(project "Shutdown"
 				(path "/624b8e71-6fec-49ba-b7c9-b659e140fc2f/2f9ac893-2047-438f-af87-5654fc0cb14f"
-					(reference "#PWR075")
+					(reference "#PWR037")
 					(unit 1)
 				)
 				(path "/624b8e71-6fec-49ba-b7c9-b659e140fc2f/5fbdbc4a-acfc-4802-ab24-0d194c32f3aa"
-					(reference "#PWR081")
+					(reference "#PWR040")
 					(unit 1)
 				)
@@
 				)
 				(path "/624b8e71-6fec-49ba-b7c9-b659e140fc2f/5fbdbc4a-acfc-4802-ab24-0d194c32f3aa"
-					(reference "Q16")
+					(reference "Q14")
 					(unit 1)
 				)
@@
 		(on_board yes)
 		(dnp no)
-		(property "Reference" "#PWR076"
+		(property "Reference" "#PWR038"
 			(at 167.64 148.59 0)
 			(effects
@@
 			(project "Shutdown"
 				(path "/624b8e71-6fec-49ba-b7c9-b659e140fc2f/2f9ac893-2047-438f-af87-5654fc0cb14f"
-					(reference "#PWR076")
+					(reference "#PWR038")
 					(unit 1)
 				)
 				(path "/624b8e71-6fec-49ba-b7c9-b659e140fc2f/5fbdbc4a-acfc-4802-ab24-0d194c32f3aa"
-					(reference "#PWR082")
-					(unit 1)
-				)
+					(reference "#PWR041")
+					(unit 1)
+				)

Commit message: Finished shutdown, 0 drc, need to export gerbers
Parts:
- renumbered D16 to D21, D17 to D22, D18 to D23, D19 to D24, R32 to R37, R33 to R38, R34 to R39, R35 to R40, R36 to R41, R37 to R42
Changed lines of the file:
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@@
 		(on_board yes)
 		(dnp no)
-		(property "Reference" "R35"
+		(property "Reference" "R40"
 			(at 184.7056 147.6295 90)
 			(effects
@@
 			(project "Shutdown"
 				(path "/624b8e71-6fec-49ba-b7c9-b659e140fc2f/2f9ac893-2047-438f-af87-5654fc0cb14f"
-					(reference "R35")
+					(reference "R40")
 					(unit 1)
 				)
 				(path "/624b8e71-6fec-49ba-b7c9-b659e140fc2f/5fbdbc4a-acfc-4802-ab24-0d194c32f3aa"
-					(reference "R41")
+					(reference "R46")
 					(unit 1)
 				)
@@
 		(on_board yes)
 		(dnp no)
-		(property "Reference" "R37"
+		(property "Reference" "R42"
 			(at 222.8921 170.8631 90)
 			(effects
@@
 			(project "Shutdown"
 				(path "/624b8e71-6fec-49ba-b7c9-b659e140fc2f/2f9ac893-2047-438f-af87-5654fc0cb14f"
-					(reference "R37")
+					(reference "R42")
 					(unit 1)
 				)
 				(path "/624b8e71-6fec-49ba-b7c9-b659e140fc2f/5fbdbc4a-acfc-4802-ab24-0d194c32f3aa"
-					(reference "R43")
+					(reference "R48")
 					(unit 1)
 				)
@@
 		(on_board yes)
 		(dnp no)
-		(property "Reference" "D18"
+		(property "Reference" "D23"
 			(at 235.5885 145.2833 90)
 			(effects
@@
 			(project "Shutdown"
 				(path "/624b8e71-6fec-49ba-b7c9-b659e140fc2f/2f9ac893-2047-438f-af87-5654fc0cb14f"
-					(reference "D18")
+					(reference "D23")
 					(unit 1)
 				)
 				(path "/624b8e71-6fec-49ba-b7c9-b659e140fc2f/5fbdbc4a-acfc-4802-ab24-0d194c32f3aa"
-					(reference "D22")
+					(reference "D27")
 					(unit 1)
 				)
@@
 		(on_board yes)
 		(dnp no)
-		(property "Reference" "#PWR039"
+		(property "Reference" "#PWR044"
 			(at 220.98 189.23 0)
 			(effects
@@
 			(project "Shutdown"
 				(path "/624b8e71-6fec-49ba-b7c9-b659e140fc2f/2f9ac893-2047-438f-af87-5654fc0cb14f"
-					(reference "#PWR039")
+					(reference "#PWR044")
 					(unit 1)
 				)
 				(path "/624b8e71-6fec-49ba-b7c9-b659e140fc2f/5fbdbc4a-acfc-4802-ab24-0d194c32f3aa"
-					(reference "#PWR042")
+					(reference "#PWR047")
 					(unit 1)
 				)
@@
 		(on_board yes)
 		(dnp no)
-		(property "Reference" "R32"
+		(property "Reference" "R37"
 			(at 222.588 131.7328 90)
 			(effects
@@
 			(project "Shutdown"
 				(path "/624b8e71-6fec-49ba-b7c9-b659e140fc2f/2f9ac893-2047-438f-af87-5654fc0cb14f"
-					(reference "R32")
+					(reference "R37")
 					(unit 1)
 				)
 				(path "/624b8e71-6fec-49ba-b7c9-b659e140fc2f/5fbdbc4a-acfc-4802-ab24-0d194c32f3aa"
-					(reference "R38")
+					(reference "R43")
 					(unit 1)
 				)
@@
 		(on_board yes)
 		(dnp no)
-		(property "Reference" "R36"
+		(property "Reference" "R41"
 			(at 201.804 162.8047 0)
 			(effects
@@
 			(project "Shutdown"
 				(path "/624b8e71-6fec-49ba-b7c9-b659e140fc2f/2f9ac893-2047-438f-af87-5654fc0cb14f"
-					(reference "R36")
+					(reference "R41")
 					(unit 1)
 				)
 				(path "/624b8e71-6fec-49ba-b7c9-b659e140fc2f/5fbdbc4a-acfc-4802-ab24-0d194c32f3aa"
-					(reference "R42")
+					(reference "R47")
 					(unit 1)
 				)
@@
 		(on_board yes)
 		(dnp no)
-		(property "Reference" "R33"
+		(property "Reference" "R38"
 			(at 234.018 131.7328 90)
 			(effects
@@
 			(project "Shutdown"
 				(path "/624b8e71-6fec-49ba-b7c9-b659e140fc2f/2f9ac893-2047-438f-af87-5654fc0cb14f"
-					(reference "R33")
+					(reference "R38")
 					(unit 1)
 				)
 				(path "/624b8e71-6fec-49ba-b7c9-b659e140fc2f/5fbdbc4a-acfc-4802-ab24-0d194c32f3aa"
-					(reference "R39")
+					(reference "R44")
 					(unit 1)
 				)
@@
 		(on_board yes)
 		(dnp no)
-		(property "Reference" "R34"
+		(property "Reference" "R39"
 			(at 169.4656 147.6295 90)
 			(effects
@@
 			(project "Shutdown"
 				(path "/624b8e71-6fec-49ba-b7c9-b659e140fc2f/2f9ac893-2047-438f-af87-5654fc0cb14f"
-					(reference "R34")
+					(reference "R39")
 					(unit 1)
 				)
 				(path "/624b8e71-6fec-49ba-b7c9-b659e140fc2f/5fbdbc4a-acfc-4802-ab24-0d194c32f3aa"
-					(reference "R40")
+					(reference "R45")
 					(unit 1)
 				)
@@
 		(on_board yes)
 		(dnp no)
-		(property "Reference" "D16"
+		(property "Reference" "D21"
 			(at 182.784 128.0941 90)
 			(effects
@@
 			(project "Shutdown"
 				(path "/624b8e71-6fec-49ba-b7c9-b659e140fc2f/2f9ac893-2047-438f-af87-5654fc0cb14f"
-					(reference "D16")
+					(reference "D21")
 					(unit 1)
 				)
 				(path "/624b8e71-6fec-49ba-b7c9-b659e140fc2f/5fbdbc4a-acfc-4802-ab24-0d194c32f3aa"
-					(reference "D20")
+					(reference "D25")
 					(unit 1)
 				)
@@
 		(on_board yes)
 		(dnp no)
-		(property "Reference" "D19"
+		(property "Reference" "D24"
 			(at 213.0765 169.2859 0)
 			(effects
@@
 			(project "Shutdown"
 				(path "/624b8e71-6fec-49ba-b7c9-b659e140fc2f/2f9ac893-2047-438f-af87-5654fc0cb14f"
-					(reference "D19")
+					(reference "D24")
 					(unit 1)
 				)
 				(path "/624b8e71-6fec-49ba-b7c9-b659e140fc2f/5fbdbc4a-acfc-4802-ab24-0d194c32f3aa"
-					(reference "D23")
+					(reference "D28")
 					(unit 1)
 				)
@@
 		(on_board yes)
 		(dnp no)
-		(property "Reference" "D17"
+		(property "Reference" "D22"
 			(at 224.1585 145.2833 90)
 			(effects
@@
 			(project "Shutdown"
 				(path "/624b8e71-6fec-49ba-b7c9-b659e140fc2f/2f9ac893-2047-438f-af87-5654fc0cb14f"
-					(reference "D17")
+					(reference "D22")
 					(unit 1)
 				)
 				(path "/624b8e71-6fec-49ba-b7c9-b659e140fc2f/5fbdbc4a-acfc-4802-ab24-0d194c32f3aa"
-					(reference "D21")
+					(reference "D26")
 					(unit 1)
 				)
@@
 		(on_board yes)
 		(dnp no)
-		(property "Reference" "#PWR037"
+		(property "Reference" "#PWR042"
 			(at 220.98 129.54 0)
 			(effects
@@
 			(project "Shutdown"
 				(path "/624b8e71-6fec-49ba-b7c9-b659e140fc2f/2f9ac893-2047-438f-af87-5654fc0cb14f"
-					(reference "#PWR037")
+					(reference "#PWR042")
 					(unit 1)
 				)
 				(path "/624b8e71-6fec-49ba-b7c9-b659e140fc2f/5fbdbc4a-acfc-4802-ab24-0d194c32f3aa"
-					(reference "#PWR040")
+					(reference "#PWR045")
 					(unit 1)
 				)
@@
 		(on_board yes)
 		(dnp no)
-		(property "Reference" "#PWR038"
+		(property "Reference" "#PWR043"
 			(at 167.64 148.59 0)
 			(effects
@@
 			(project "Shutdown"
 				(path "/624b8e71-6fec-49ba-b7c9-b659e140fc2f/2f9ac893-2047-438f-af87-5654fc0cb14f"
-					(reference "#PWR038")
+					(reference "#PWR043")
 					(unit 1)
 				)
 				(path "/624b8e71-6fec-49ba-b7c9-b659e140fc2f/5fbdbc4a-acfc-4802-ab24-0d194c32f3aa"
-					(reference "#PWR041")
-					(unit 1)
-				)
+					(reference "#PWR046")
+					(unit 1)
+				)

Commit message: schematic updated to V2 extra crispy
Parts:
- removed D22, D23: Red, LED_SMD:LED_0805_2012Metric, symbol -Diodes-LED:NCD0805R1
- removed R37, R38: 510, Resistor_SMD:R_0603_1608Metric_Pad0.98x0.95mm_HandSolder, symbol -R-SMD-0603:R-0603-510-1%-100mW-100PPM
- removed R42: 51, Resistor_SMD:R_0603_1608Metric_Pad0.98x0.95mm_HandSolder, symbol -R-SMD-0603:R-0603-51-1%-100mW-100PPM
- added D27, D28: Red, LED_SMD:LED_0805_2012Metric, symbol -Diodes-LED:NCD0805R1
- added R37: 1M, Resistor_SMD:R_0603_1608Metric_Pad0.98x0.95mm_HandSolder, symbol -R-SMD-0603:R-0603-1M-1%-100mW-100PPM
- added R38, R39: 680, Resistor_SMD:R_0603_1608Metric_Pad0.98x0.95mm_HandSolder, symbol -R-SMD-0603:R-0603-680-1%-100mW-100PPM
- renumbered D21 to D26, D24 to D29, R39 to R41, R41 to R42
Connections:
- net BATT+PROT: now also R38.2, R39.2
- net GND: now also D29.2 (A), Q13.2 (S), R37.1
- net OUTPUT: now also R37.2
- net at Q13.3 (D): now also D27.1 (K), D28.1 (K)
- new net: D27.2 (A), R38.1
- new net: D28.2 (A), R39.1
Other:
- moved on the sheet: D26, D29, Q12, Q13, R40, R41, R42

Commit message: layout done extra crispy v2
Changed lines of the file:
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@@
 	(text_box "NOTE: The 1M pulldown resistor here so the Source of the next fault stage (BMS after BSPD for example) goes to 0V, ensuring the output is not floating (which could float to 12V)."
 		(exclude_from_sim no)
-		(at 194.31 118.3606 0)
-		(size 26.67 14.9894)
+		(at 194.31 118.11 0)
+		(size 26.67 15.24)
 		(margins 0.9525 0.9525 0.9525 0.9525)
 		(stroke
