File: Shutdown.kicad_pcb (KiCad board)
At the start: 4 copper layers, 178.3 x 67.6 mm, 8 parts, among them J1 0194270049, J2 0194270049, Q24 AO3400A

Commit message: Finished shutdown, 0 drc, need to export gerbers
Parts:
- removed the G*** at (203.1, 126.9)
- added BMS1: ~, TestPoint:TestPoint_Pad_1.0x1.0mm, F.Cu at (126.7, 112.5)
- added BOTS1: BOTS, TestPoint:TestPoint_Pad_1.0x1.0mm, F.Cu at (205.3, 115.9)
- added BSPD1: ~, TestPoint:TestPoint_Pad_1.0x1.0mm, F.Cu at (114.4, 109.3)
- added BYPASS1: ~, TestPoint:TestPoint_Pad_1.0x1.0mm, F.Cu at (165.4, 116.7)
- added C1: 470nF, Capacitor_SMD:C_0603_1608Metric_Pad1.08x0.95mm_HandSolder, F.Cu at (147.3, 130.9)
- added C2: 100nF, Capacitor_SMD:C_0603_1608Metric_Pad1.08x0.95mm_HandSolder, F.Cu at (148.1, 135.3)
- added CS1: CS, TestPoint:TestPoint_Pad_1.0x1.0mm, F.Cu at (193.8, 115.9)
- added D1: Blue, LED_SMD:LED_0805_2012Metric, F.Cu at (231.2, 112.7)
- added D10: Blue, LED_SMD:LED_0805_2012Metric, B.Cu at (256.5, 112.7)
- added D11: BZT52C16, Diode_SMD:D_SOD-123, F.Cu at (217.6, 142.2)
- added D12: Green, LED_SMD:LED_0805_2012Metric, F.Cu at (240.8, 129.5)
- added D13: Green, LED_SMD:LED_0805_2012Metric, B.Cu at (240.8, 129.5)
- added D14: Green, LED_SMD:LED_0805_2012Metric, F.Cu at (253.9, 129.6)
- added D15: Green, LED_SMD:LED_0805_2012Metric, B.Cu at (253.9, 129.6)
- added D16: BZT52C16, Diode_SMD:D_SOD-123, F.Cu at (161.5, 123.4)
- added D17: BZT52C16, Diode_SMD:D_SOD-123, F.Cu at (146.6, 116.0)
- added D18: BZT52C16, Diode_SMD:D_SOD-123, F.Cu at (155.6, 127.2)
- added D19: BZT52C16, Diode_SMD:D_SOD-123, F.Cu at (161.3, 130.7)
- added D2: Blue, LED_SMD:LED_0805_2012Metric, B.Cu at (231.2, 112.7)
- added D20: BZT52C16, Diode_SMD:D_SOD-123, F.Cu at (147.9, 126.0)
- added D21: BZT52C16, Diode_SMD:D_SOD-123, F.Cu at (116.1, 113.8)
- added D22: Red, LED_SMD:LED_0805_2012Metric, F.Cu at (123.6, 125.6)
- added D23: Red, LED_SMD:LED_0805_2012Metric, B.Cu at (123.6, 125.6)
- added D24: BZT52C16, Diode_SMD:D_SOD-123, F.Cu at (119.1, 119.1)
- added D25: BZT52C16, Diode_SMD:D_SOD-123, F.Cu at (133.0, 113.5)
- added D26: Red, LED_SMD:LED_0805_2012Metric, F.Cu at (140.4, 125.3)
- added D27: Red, LED_SMD:LED_0805_2012Metric, B.Cu at (140.4, 125.3)
- added D28: BZT52C16, Diode_SMD:D_SOD-123, F.Cu at (136.0, 118.8)
- added D29: BZT52C16, Diode_SMD:D_SOD-123, F.Cu at (128.6, 134.6)
- added D3: Red, LED_SMD:LED_0805_2012Metric, F.Cu at (212.7, 105.5)
- added D30: BZT52C16, Diode_SMD:D_SOD-123, F.Cu at (128.6, 140.0)
- added D31: BZT52C16, Diode_SMD:D_SOD-123, F.Cu at (173.3, 115.8)
- added D32: BZT52C16, Diode_SMD:D_SOD-123, F.Cu at (188.1, 115.8)
- added D33: BZT52C16, Diode_SMD:D_SOD-123, F.Cu at (199.8, 115.8)
- added D34: BZT52C16, Diode_SMD:D_SOD-123, F.Cu at (211.6, 115.8)
- added D35: Red, LED_SMD:LED_0805_2012Metric, F.Cu at (222.0, 125.8)
- added D36: Red, LED_SMD:LED_0805_2012Metric, B.Cu at (222.0, 125.8)
- added D37: Red, LED_SMD:LED_0805_2012Metric, F.Cu at (171.4, 125.5)
- added D38: Red, LED_SMD:LED_0805_2012Metric, B.Cu at (171.4, 125.5)
- added D39: Red, LED_SMD:LED_0805_2012Metric, F.Cu at (186.2, 125.5)
- added D4: Red, LED_SMD:LED_0805_2012Metric, B.Cu at (212.6, 105.5)
- added D40: Red, LED_SMD:LED_0805_2012Metric, B.Cu at (186.2, 125.5)
- added D41: Red, LED_SMD:LED_0805_2012Metric, F.Cu at (197.9, 125.5)
- added D42: Red, LED_SMD:LED_0805_2012Metric, B.Cu at (197.9, 125.5)
- added D43: Red, LED_SMD:LED_0805_2012Metric, F.Cu at (209.7, 125.5)
- added D44: Red, LED_SMD:LED_0805_2012Metric, B.Cu at (209.7, 125.5)
- added D45: BZT52C16, Diode_SMD:D_SOD-123, F.Cu at (110.0, 109.8)
- added D46: BZT52C16, Diode_SMD:D_SOD-123, F.Cu at (104.6, 110.1)
- added D47: BZT52C16, Diode_SMD:D_SOD-123, F.Cu at (103.6, 121.4)
- added D48: Red, LED_SMD:LED_0805_2012Metric, F.Cu at (104.5, 124.9)
- added D49: Red, LED_SMD:LED_0805_2012Metric, B.Cu at (104.6, 124.9)
- added D5: Red, LED_SMD:LED_0805_2012Metric, F.Cu at (221.5, 105.7)
- added D6: Red, LED_SMD:LED_0805_2012Metric, B.Cu at (221.5, 105.7)
- added D7: Blue, LED_SMD:LED_0805_2012Metric, F.Cu at (244.0, 112.7)
- added D8: Blue, LED_SMD:LED_0805_2012Metric, B.Cu at (244.0, 112.7)
- added D9: Blue, LED_SMD:LED_0805_2012Metric, F.Cu at (256.5, 112.7)
- added G***: LOGO, LOGO, B.Cu at (114.9, 104.5)
- added G***: LOGO, LOGO, B.Cu at (136.8, 104.8)
- added HVILS1: HVILS, TestPoint:TestPoint_Pad_1.0x1.0mm, F.Cu at (178.9, 115.7)
- added IMD1: ~, TestPoint:TestPoint_Pad_1.0x1.0mm, F.Cu at (153.4, 120.4)
- added Q1: AO3400A, Package_TO_SOT_SMD:SOT-23, F.Cu at (232.1, 109.2)
- added Q10: SI2318CDS-T1-GE3, Package_TO_SOT_SMD:SOT-23-3, F.Cu at (159.0, 127.6)
- added Q11: SI2347DS-T1-GE3, Package_TO_SOT_SMD:SOT-23-3, F.Cu at (151.3, 125.3)
- added Q12: SI2347DS-T1-GE3, Package_TO_SOT_SMD:SOT-23-3, F.Cu at (116.0, 117.3)
- added Q13: SI2318CDS-T1-GE3, Package_TO_SOT_SMD:SOT-23-3, F.Cu at (122.5, 119.9)
- added Q14: SI2347DS-T1-GE3, Package_TO_SOT_SMD:SOT-23-3, F.Cu at (132.8, 117.0)
- added Q15: SI2318CDS-T1-GE3, Package_TO_SOT_SMD:SOT-23-3, F.Cu at (139.4, 119.6)
- added Q16: SI2347DS-T1-GE3, Package_TO_SOT_SMD:SOT-23-3, F.Cu at (132.1, 134.7)
- added Q17: SI2347DS-T1-GE3, Package_TO_SOT_SMD:SOT-23-3, F.Cu at (132.1, 140.1)
- added Q18: SI2347DS-T1-GE3, Package_TO_SOT_SMD:SOT-23-3, F.Cu at (173.3, 119.3)
- added Q19: SI2347DS-T1-GE3, Package_TO_SOT_SMD:SOT-23-3, F.Cu at (188.1, 119.3)
- added Q2: AO3400A, Package_TO_SOT_SMD:SOT-23, F.Cu at (244.9, 109.2)
- added Q20: SI2347DS-T1-GE3, Package_TO_SOT_SMD:SOT-23-3, F.Cu at (199.8, 119.3)
- added Q21: SI2347DS-T1-GE3, Package_TO_SOT_SMD:SOT-23-3, F.Cu at (211.6, 119.3)
- added Q22: SI2347DS-T1-GE3, Package_TO_SOT_SMD:SOT-23-3, F.Cu at (109.2, 105.5)
- added Q23: SI2318CDS-T1-GE3, Package_TO_SOT_SMD:SOT-23-3, F.Cu at (104.5, 113.1)
- added Q3: AO3400A, Package_TO_SOT_SMD:SOT-23, F.Cu at (257.4, 109.2)
- added Q4: SI2347DS-T1-GE3, Package_TO_SOT_SMD:SOT-23-3, F.Cu at (223.1, 142.9)
- added Q5: AO3400A, Package_TO_SOT_SMD:SOT-23, F.Cu at (239.8, 125.8)
- added Q6: AO3400A, Package_TO_SOT_SMD:SOT-23, F.Cu at (252.8, 126.1)
- added Q7: SI2347DS-T1-GE3, Package_TO_SOT_SMD:SOT-23-3, F.Cu at (159.2, 120.3)
- added Q8: SI2318CDS-T1-GE3, Package_TO_SOT_SMD:SOT-23-3, F.Cu at (142.9, 116.2)
- added Q9: SI2318CDS-T1-GE3, Package_TO_SOT_SMD:SOT-23-3, F.Cu at (158.0, 124.0)
- added R1: 22, Resistor_SMD:R_0603_1608Metric_Pad0.98x0.95mm_HandSolder, F.Cu at (229.3, 109.1)
- added R10: 510, Resistor_SMD:R_0603_1608Metric_Pad0.98x0.95mm_HandSolder, F.Cu at (219.4, 105.6)
- added R11: 510, Resistor_SMD:R_0603_1608Metric_Pad0.98x0.95mm_HandSolder, B.Cu at (219.4, 105.6)
- added R12: 100k, Resistor_SMD:R_0603_1608Metric_Pad0.98x0.95mm_HandSolder, F.Cu at (214.6, 142.1)
- added R13: 2.2k, Resistor_SMD:R_0603_1608Metric_Pad0.98x0.95mm_HandSolder, F.Cu at (233.2, 112.7)
- added R14: 2.2k, Resistor_SMD:R_0603_1608Metric_Pad0.98x0.95mm_HandSolder, B.Cu at (233.2, 112.7)
- added R15: 2.2k, Resistor_SMD:R_0603_1608Metric_Pad0.98x0.95mm_HandSolder, F.Cu at (246.0, 112.7)
- added R16: 2.2k, Resistor_SMD:R_0603_1608Metric_Pad0.98x0.95mm_HandSolder, B.Cu at (246.0, 112.7)
- added R17: 2.2k, Resistor_SMD:R_0603_1608Metric_Pad0.98x0.95mm_HandSolder, F.Cu at (258.5, 112.7)
- added R18: 2.2k, Resistor_SMD:R_0603_1608Metric_Pad0.98x0.95mm_HandSolder, B.Cu at (258.5, 112.7)
- added R19: 10k, Resistor_SMD:R_0603_1608Metric_Pad0.98x0.95mm_HandSolder, F.Cu at (220.1, 141.0)
- added R2: 22, Resistor_SMD:R_0603_1608Metric_Pad0.98x0.95mm_HandSolder, F.Cu at (242.1, 109.1)
- added R20: 22, Resistor_SMD:R_0603_1608Metric_Pad0.98x0.95mm_HandSolder, F.Cu at (237.0, 125.8)
- added R21: 22, Resistor_SMD:R_0603_1608Metric_Pad0.98x0.95mm_HandSolder, F.Cu at (249.9, 126.0)
- added R22: 100k, Resistor_SMD:R_0603_1608Metric_Pad0.98x0.95mm_HandSolder, F.Cu at (237.3, 123.2)
- added R23: 100k, Resistor_SMD:R_0603_1608Metric_Pad0.98x0.95mm_HandSolder, F.Cu at (250.2, 123.5)
- added R24: 5.1k, Resistor_SMD:R_0603_1608Metric_Pad0.98x0.95mm_HandSolder, F.Cu at (238.8, 129.4)
- added R25: 5.1k, Resistor_SMD:R_0603_1608Metric_Pad0.98x0.95mm_HandSolder, B.Cu at (238.8, 129.4)
- added R26: 5.1k, Resistor_SMD:R_0603_1608Metric_Pad0.98x0.95mm_HandSolder, F.Cu at (251.8, 129.6)
- added R27: 5.1k, Resistor_SMD:R_0603_1608Metric_Pad0.98x0.95mm_HandSolder, B.Cu at (251.8, 129.6)
- added R28: 100k, Resistor_SMD:R_0603_1608Metric_Pad0.98x0.95mm_HandSolder, F.Cu at (166.8, 127.3)
- added R29: 100k, Resistor_SMD:R_0603_1608Metric_Pad0.98x0.95mm_HandSolder, F.Cu at (162.9, 127.3)
- added R3: 22, Resistor_SMD:R_0603_1608Metric_Pad0.98x0.95mm_HandSolder, F.Cu at (254.6, 109.1)
- added R30: 100k, Resistor_SMD:R_0603_1608Metric_Pad0.98x0.95mm_HandSolder, F.Cu at (163.7, 124.6)
- added R31: 100, Resistor_SMD:R_0603_1608Metric_Pad0.98x0.95mm_HandSolder, F.Cu at (147.5, 119.5)
- added R32: 2.2k, Resistor_SMD:R_0603_1608Metric_Pad0.98x0.95mm_HandSolder, F.Cu at (147.5, 121.1)
- added R33: 100k, Resistor_SMD:R_0603_1608Metric_Pad0.98x0.95mm_HandSolder, F.Cu at (154.1, 123.8)
- added R34: 100k, Resistor_SMD:R_0603_1608Metric_Pad0.98x0.95mm_HandSolder, F.Cu at (153.3, 127.7)
- added R35: 100k, Resistor_SMD:R_0603_1608Metric_Pad0.98x0.95mm_HandSolder, F.Cu at (150.7, 127.8)
- added R36: 390k, Resistor_SMD:R_0603_1608Metric_Pad0.98x0.95mm_HandSolder, F.Cu at (147.2, 129.2)
- added R37: 510, Resistor_SMD:R_0603_1608Metric_Pad0.98x0.95mm_HandSolder, F.Cu at (121.6, 125.6)
- added R38: 510, Resistor_SMD:R_0603_1608Metric_Pad0.98x0.95mm_HandSolder, B.Cu at (121.6, 125.6)
- added R39: 100k, Resistor_SMD:R_0603_1608Metric_Pad0.98x0.95mm_HandSolder, F.Cu at (120.5, 112.2)
- added R4: 10k, Resistor_SMD:R_0603_1608Metric_Pad0.98x0.95mm_HandSolder, F.Cu at (229.6, 106.6)
- added R40: 100k, Resistor_SMD:R_0603_1608Metric_Pad0.98x0.95mm_HandSolder, F.Cu at (120.5, 113.8)
- added R41: 100k, Resistor_SMD:R_0603_1608Metric_Pad0.98x0.95mm_HandSolder, F.Cu at (121.4, 116.3)
- added R42: 51, Resistor_SMD:R_0603_1608Metric_Pad0.98x0.95mm_HandSolder, F.Cu at (118.2, 122.4)
- added R43: 510, Resistor_SMD:R_0603_1608Metric_Pad0.98x0.95mm_HandSolder, F.Cu at (138.5, 125.3)
- added R44: 510, Resistor_SMD:R_0603_1608Metric_Pad0.98x0.95mm_HandSolder, B.Cu at (138.5, 125.3)
- added R45: 100k, Resistor_SMD:R_0603_1608Metric_Pad0.98x0.95mm_HandSolder, F.Cu at (137.3, 111.9)
- added R46: 100k, Resistor_SMD:R_0603_1608Metric_Pad0.98x0.95mm_HandSolder, F.Cu at (137.3, 113.5)
- added R47: 100k, Resistor_SMD:R_0603_1608Metric_Pad0.98x0.95mm_HandSolder, F.Cu at (138.2, 116.0)
- added R48: 51, Resistor_SMD:R_0603_1608Metric_Pad0.98x0.95mm_HandSolder, F.Cu at (135.1, 122.1)
- added R49: 100k, Resistor_SMD:R_0603_1608Metric_Pad0.98x0.95mm_HandSolder, F.Cu at (135.3, 134.6)
- added R5: 10k, Resistor_SMD:R_0603_1608Metric_Pad0.98x0.95mm_HandSolder, F.Cu at (242.4, 106.6)
- added R50: 100k, Resistor_SMD:R_0603_1608Metric_Pad0.98x0.95mm_HandSolder, F.Cu at (135.3, 140.0)
- added R51: 100k, Resistor_SMD:R_0603_1608Metric_Pad0.98x0.95mm_HandSolder, F.Cu at (134.2, 142.7)
- added R52: 510, Resistor_SMD:R_0603_1608Metric_Pad0.98x0.95mm_HandSolder, F.Cu at (223.9, 125.7)
- added R53: 510, Resistor_SMD:R_0603_1608Metric_Pad0.98x0.95mm_HandSolder, B.Cu at (223.9, 125.7)
- added R54: 100k, Resistor_SMD:R_0603_1608Metric_Pad0.98x0.95mm_HandSolder, F.Cu at (170.6, 119.1)
- added R55: 100k, Resistor_SMD:R_0603_1608Metric_Pad0.98x0.95mm_HandSolder, F.Cu at (178.0, 118.2)
- added R56: 100k, Resistor_SMD:R_0603_1608Metric_Pad0.98x0.95mm_HandSolder, F.Cu at (192.7, 118.2)
- added R57: 100k, Resistor_SMD:R_0603_1608Metric_Pad0.98x0.95mm_HandSolder, F.Cu at (204.4, 118.2)
- added R58: 100k, Resistor_SMD:R_0603_1608Metric_Pad0.98x0.95mm_HandSolder, F.Cu at (216.4, 118.5)
- added R59: 1M, Resistor_SMD:R_0603_1608Metric_Pad0.98x0.95mm_HandSolder, F.Cu at (185.3, 119.1)
- added R6: 10k, Resistor_SMD:R_0603_1608Metric_Pad0.98x0.95mm_HandSolder, F.Cu at (254.9, 106.6)
- added R60: 100k, Resistor_SMD:R_0603_1608Metric_Pad0.98x0.95mm_HandSolder, F.Cu at (197.1, 119.1)
- added R61: 100k, Resistor_SMD:R_0603_1608Metric_Pad0.98x0.95mm_HandSolder, F.Cu at (208.9, 119.1)
- added R62: 100k, Resistor_SMD:R_0603_1608Metric_Pad0.98x0.95mm_HandSolder, F.Cu at (220.7, 119.6)
- added R63: 510, Resistor_SMD:R_0603_1608Metric_Pad0.98x0.95mm_HandSolder, F.Cu at (173.4, 125.5)
- added R64: 510, Resistor_SMD:R_0603_1608Metric_Pad0.98x0.95mm_HandSolder, B.Cu at (173.4, 125.5)
- added R65: 510, Resistor_SMD:R_0603_1608Metric_Pad0.98x0.95mm_HandSolder, F.Cu at (188.1, 125.5)
- added R66: 510, Resistor_SMD:R_0603_1608Metric_Pad0.98x0.95mm_HandSolder, B.Cu at (188.1, 125.5)
- added R67: 510, Resistor_SMD:R_0603_1608Metric_Pad0.98x0.95mm_HandSolder, F.Cu at (199.8, 125.5)
- added R68: 510, Resistor_SMD:R_0603_1608Metric_Pad0.98x0.95mm_HandSolder, B.Cu at (199.8, 125.5)
- added R69: 510, Resistor_SMD:R_0603_1608Metric_Pad0.98x0.95mm_HandSolder, F.Cu at (211.6, 125.5)
- added R7: 0, Resistor_SMD:R_0603_1608Metric_Pad0.98x0.95mm_HandSolder, F.Cu at (214.6, 143.8)
- added R70: 510, Resistor_SMD:R_0603_1608Metric_Pad0.98x0.95mm_HandSolder, B.Cu at (211.6, 125.5)
- added R71: 10k, Resistor_SMD:R_0603_1608Metric_Pad0.98x0.95mm_HandSolder, F.Cu at (107.8, 114.0)
- added R72: 100, Resistor_SMD:R_0603_1608Metric_Pad0.98x0.95mm_HandSolder, F.Cu at (109.5, 114.0)
- added R73: 100, Resistor_SMD:R_0603_1608Metric_Pad0.98x0.95mm_HandSolder, F.Cu at (99.7, 114.8)
- added R74: 1M, Resistor_SMD:R_0603_1608Metric_Pad0.98x0.95mm_HandSolder, F.Cu at (101.3, 114.8)
- added R75: 100, Resistor_SMD:R_0603_1608Metric_Pad0.98x0.95mm_HandSolder, F.Cu at (101.3, 118.2)
- added R76: 510, Resistor_SMD:R_0603_1608Metric_Pad0.98x0.95mm_HandSolder, F.Cu at (102.7, 125.0)
- added R77: 510, Resistor_SMD:R_0603_1608Metric_Pad0.98x0.95mm_HandSolder, B.Cu at (102.7, 125.0)
- added R8: 510, Resistor_SMD:R_0603_1608Metric_Pad0.98x0.95mm_HandSolder, F.Cu at (210.7, 105.6)
- added R9: 510, Resistor_SMD:R_0603_1608Metric_Pad0.98x0.95mm_HandSolder, B.Cu at (210.7, 105.6)
- added TSMS1: TSMS, TestPoint:TestPoint_Pad_1.0x1.0mm, F.Cu at (220.6, 116.3)
- added U1: TSB712AIDT, Package_SO:SOIC-8_5.3x5.3mm_P1.27mm, F.Cu at (142.4, 138.1)
- added VIN1: ~, TestPoint:TestPoint_Pad_1.0x1.0mm, F.Cu at (214.9, 139.8)
- Q24: value AO3400A -> SI2347DS-T1-GE3
- moved Q24 155.0 mm to (104.3, 118.2), turned to 180 degrees
- turned J1 to 180 degrees
- turned J2 to 180 degrees
Connections:
- Q24 pad 2: Net-(Q24-S) -> BATT+PROT
- Q24 pad 3: BATT+PROT -> Net-(D47-A)
Routing:
- net /BYPASS-BTN: track 0.00 -> 129.6 mm, vias 0 -> 3
- net /TSSI-STATUS: track 0.00 -> 120.3 mm
- net /SD-POWER: track 0.00 -> 102.4 mm, vias 0 -> 3
- net /BOTS-B: track 0.00 -> 98.8 mm
- net /BOTS-A: track 0.00 -> 88.1 mm
- net /HVILS-A: track 0.00 -> 86.6 mm, vias 0 -> 2
- net /CRASH-SW-A: track 0.00 -> 85.9 mm
- net GND: track 0.00 -> 78.8 mm, vias 0 -> 32
- net /NEG-AIRS-DEBUG: track 0.00 -> 67.8 mm, vias 0 -> 1
- net /BMS-FAULT: track 0.00 -> 63.9 mm, vias 0 -> 2
- net /POS-AIRS-DEBUG: track 0.00 -> 58.6 mm, vias 0 -> 1
- net BATT+: track 0.00 -> 56.6 mm, vias 0 -> 3
- net /TRACTIVE-FAN-ON: track 0.00 -> 56.0 mm
- net /PRECHARGE-DEBUG: track 0.00 -> 55.7 mm, vias 0 -> 1
- net BATT+PROT: track 0.00 -> 54.3 mm, vias 0 -> 35
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- added copper zone on In2.Cu, net BATT+PROT
- added copper zone on B.Cu, net GND
- added copper zone on F.Cu, net GND
Other:
- board text added: "ACCY FAN"
- board text added: "AIR+ RELAY"
- board text added: "AIR- RELAY"
- board text added: "BATT+"
- board text added: "BMS FAULT"
- board text added: "BOTS SWITCH"
- board text added: "BSPD FAULT"
- board text added: "BYPASS"
- board text added: "CRASH SWITCH"
- board text added: "DEBUG LIGHTS"
- board text added: "HVILS"
- board text added: "IMD FAULT"
- board text added: "MK.11 Shutdown V1"
- board text added: "PRECHG RELAY"
- board text added: "SHUTDOWN POWER"
- board text added: "TRACTIVE FAN"
- board text added: "TSMS"
- board text removed: "MK11 SHUTDOWN V1"
- board text removed: "MK11 Shutdown V1 Drive Documentation"

Commit message: EXPORTED Gerbers, fixed qr code
Parts:
- moved G*** 1.05 mm to (137.0, 103.8)
