File: Shutdown.kicad_pcb (KiCad board)
At the start: 4 copper layers, 178.3 x 67.6 mm, 170 parts, among them J1 0194270049, J2 0194270049, Q1 AO3400A, Q10 SI2318CDS-T1-GE3, Q11 SI2347DS-T1-GE3, Q12 SI2347DS-T1-GE3, Q13 SI2318CDS-T1-GE3, Q14 SI2347DS-T1-GE3, Q15 SI2318CDS-T1-GE3, Q16 SI2347DS-T1-GE3, Q17 SI2347DS-T1-GE3, Q18 SI2347DS-T1-GE3, Q19 SI2347DS-T1-GE3, Q2 AO3400A, Q20 SI2347DS-T1-GE3, Q21 SI2347DS-T1-GE3, Q22 SI2347DS-T1-GE3, Q23 SI2318CDS-T1-GE3, Q24 SI2347DS-T1-GE3, Q3 AO3400A, Q4 SI2347DS-T1-GE3, Q5 AO3400A, Q6 AO3400A, Q7 SI2347DS-T1-GE3, Q8 SI2318CDS-T1-GE3, Q9 SI2318CDS-T1-GE3, U1 TSB712AIDT

Commit message: schematic updated to V2 extra crispy
Parts:
- added D50: BZT52C16, Diode_SMD:D_SOD-123, F.Cu at (191.9, 222.2)
- added D51: BZT52C16, Diode_SMD:D_SOD-123, F.Cu at (205.6, 213.3)
- added D52: BZT52C16, Diode_SMD:D_SOD-123, F.Cu at (205.6, 216.6)
- added D53: BZT52C16, Diode_SMD:D_SOD-123, F.Cu at (205.6, 220.0)
- added D54: Red, LED_SMD:LED_0805_2012Metric, F.Cu at (210.7, 220.6)
- added D55: Red, LED_SMD:LED_0805_2012Metric, F.Cu at (210.7, 223.7)
- added Q25: SI2347DS-T1-GE3, Package_TO_SOT_SMD:SOT-23-3, F.Cu at (192.2, 218.3)
- added R78: 1M, Resistor_SMD:R_0603_1608Metric_Pad0.98x0.95mm_HandSolder, F.Cu at (192.6, 212.8)
- added R79: 100, Resistor_SMD:R_0603_1608Metric_Pad0.98x0.95mm_HandSolder, F.Cu at (210.7, 212.8)
- added R80: 680, Resistor_SMD:R_0603_1608Metric_Pad0.98x0.95mm_HandSolder, F.Cu at (210.7, 215.4)
- added R81: 680, Resistor_SMD:R_0603_1608Metric_Pad0.98x0.95mm_HandSolder, F.Cu at (210.7, 217.9)
- D1, D2: value Blue -> BZT52C16; footprint LED_SMD:LED_0805_2012Metric -> Diode_SMD:D_SOD-123
- D10, D7, D8, D9: value Blue -> White
- D11, D28, D31, D32, D45, D46, D47: value BZT52C16 -> Red; footprint Diode_SMD:D_SOD-123 -> LED_SMD:LED_0805_2012Metric
- D12, D13, D14: value Green -> Red
- D15: value Green -> BZT52C16; footprint LED_SMD:LED_0805_2012Metric -> Diode_SMD:D_SOD-123
- D17, D18, D19, D20, D21: value BZT52C16 -> Blue; footprint Diode_SMD:D_SOD-123 -> LED_SMD:LED_0805_2012Metric
- D22: value Red -> Blue
- D23, D26, D3, D35, D36, D37, D38, D39, D4, D5, D6: value Red -> BZT52C16; footprint LED_SMD:LED_0805_2012Metric -> Diode_SMD:D_SOD-123
- D40, D41: value Red -> Green
- Q1, Q2, Q6: value AO3400A -> SI2347DS-T1-GE3; footprint Package_TO_SOT_SMD:SOT-23 -> Package_TO_SOT_SMD:SOT-23-3
- Q11, Q22, Q4, Q7: value SI2347DS-T1-GE3 -> SI2318CDS-T1-GE3
- Q23: value SI2318CDS-T1-GE3 -> SI2347DS-T1-GE3
- Q24: value SI2347DS-T1-GE3 -> SI2318CDS-T1-GE3; footprint Package_TO_SOT_SMD:SOT-23 -> Package_TO_SOT_SMD:SOT-23-3
- Q3, Q5: value AO3400A -> SI2318CDS-T1-GE3; footprint Package_TO_SOT_SMD:SOT-23 -> Package_TO_SOT_SMD:SOT-23-3
- R1: value 22 -> 0
- R10, R11, R52, R63, R9: value 510 -> 100k
- R12: value 100k -> 390k
- R13, R14, R15, R16: value 2.2k -> 6.8k
- R17, R18: value 2.2k -> 680
- R19, R71: value 10k -> 680
- R2: value 22 -> 100k
- R20: value 22 -> 680
- R22, R33: value 100k -> 22
- R24: value 5.1k -> 100k
- R25, R26, R27: value 5.1k -> 560
- R28, R29, R30: value 100k -> 560
- R3: value 22 -> 10k
- R31: value 100 -> 22
- R32: value 2.2k -> 22
- R34, R35: value 100k -> 10k
- R36: value 390k -> 10k
- R37, R43: value 510 -> 1M
- R38, R44, R65, R66, R67, R68, R69, R70: value 510 -> 680
- R39, R45: value 100k -> 680
- R4, R5, R6: value 10k -> 100k
- R42, R48: value 51 -> 100k
- R53, R64: value 510 -> 10k
- R54, R55: value 100k -> 3.6k
- R59: value 1M -> 100k
- R60: value 100k -> 20k
- R7: value 0 -> 100
- R72: value 100 -> 680
- R73: value 100 -> 100k
- R75: value 100 -> 10k
- R76, R77: value 510 -> 100
- R8: value 510 -> 2.2k; footprint Resistor_SMD:R_0603_1608Metric_Pad0.98x0.95mm_HandSolder -> Resistor_SMD:R_2512_6332Metric_Pad1.40x3.35mm_HandSolder
- moved MH1 209.0 mm to (291.4, 185.0), turned to 180 degrees
- moved R73 200.3 mm to (292.0, 170.8), turned to -90 degrees
- moved R74 197.1 mm to (290.3, 170.8), turned to 90 degrees
- moved R75 195.2 mm to (290.3, 167.4), turned to 90 degrees
- moved D46 193.8 mm to (287.0, 175.5), turned to 180 degrees
- moved Q23 192.0 mm to (287.1, 172.5), turned to 180 degrees
- moved MH4 191.4 mm to (291.4, 146.6), turned to 180 degrees
- moved R77 189.7 mm to (289.0, 160.7), turned to -90 degrees
- moved R76 189.7 mm to (289.0, 160.7), turned to -90 degrees
- moved Q24 189.6 mm to (287.4, 167.4), turned to 0 degrees
- moved D47 189.5 mm to (288.1, 164.2), turned to 0 degrees
- moved Q22 188.6 mm to (282.4, 180.1), turned to 0 degrees
- moved D48 186.0 mm to (287.1, 160.7), turned to 90 degrees
- moved D49 186.0 mm to (287.1, 160.7), turned to 90 degrees
- moved R71 185.2 mm to (283.8, 171.6), turned to 90 degrees
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Connections:
- D11 pad 1: Net-(D11-K) -> GND
- D13 pad 1: GND -> /BYPASS-BTN
- D14 pad 1: GND -> /BYPASS-BTN
- D15 pad 1: GND -> Net-(D15-K)
- D15 pad 2: Net-(D15-A) -> GND
- D16 pad 1: /IMD-Fault-Passthru/OUTPUT -> Net-(D16-K)
- D16 pad 2: Net-(D16-A) -> GND
- D17 pad 2: GND -> Net-(D17-A)
- D18 pad 1: Net-(D18-K) -> Net-(D17-K)
- D18 pad 2: GND -> Net-(D18-A)
- D19 pad 2: GND -> Net-(D19-A)
- D2 pad 1: Net-(D2-K) -> /IMD-Fault-Passthru/OUTPUT
- D2 pad 2: Net-(D1-A) -> Net-(D2-A)
- D20 pad 1: BATT+PROT -> Net-(D19-K)
- D21 pad 1: /BMS-Fault-Passthru/INPUT -> Net-(D21-K)
- D22 pad 1: Net-(D22-K) -> Net-(D21-K)
- D23 pad 1: Net-(D22-K) -> Net-(D23-K)
- D23 pad 2: Net-(D23-A) -> GND
- D24 pad 2: Net-(D24-A) -> GND
- D25 pad 1: /BMS-Fault-Passthru/OUTPUT -> Net-(D25-K)
- D25 pad 2: Net-(D25-A) -> GND
- D26 pad 1: Net-(D26-K) -> /BMS-Fault-Passthru/INPUT
- D27 pad 1: Net-(D26-K) -> Net-(D27-K)
- D28 pad 1: Net-(D28-K) -> Net-(D27-K)
- D29 pad 1: BATT+PROT -> Net-(D29-K)
- D29 pad 2: Net-(D29-A) -> GND
- D3 pad 1: GND -> Net-(D3-K)
- D3 pad 2: Net-(D3-A) -> GND
- D30 pad 1: Net-(D30-K) -> /BMS-Fault-Passthru/OUTPUT
- D31 pad 1: /HVILS-A -> Net-(D31-K)
- D32 pad 1: /CRASH-SW-A -> Net-(D31-K)
- D33 pad 1: /BOTS-A -> Net-(D33-K)
- D33 pad 2: Net-(D33-A) -> GND
- D34 pad 1: /BOTS-B -> BATT+PROT
- D35 pad 1: GND -> Net-(D35-K)
- D36 pad 1: GND -> Net-(D36-K)
- D37 pad 1: GND -> /CRASH-SW-A
- D38 pad 1: GND -> /BOTS-A
- D39 pad 1: GND -> /BOTS-B
- D4 pad 1: GND -> Net-(D4-K)
- D4 pad 2: Net-(D4-A) -> GND
- D42 pad 1: GND -> Net-(D42-K)
- D43 pad 1: GND -> Net-(D42-K)
- D45 pad 1: BATT+PROT -> GND
- D46 pad 1: Net-(D46-K) -> GND
- D46 pad 2: GND -> Net-(D46-A)
- D47 pad 1: Net-(D47-K) -> GND
- D5 pad 1: /BYPASS-BTN -> Net-(D5-K)
- D5 pad 2: Net-(D5-A) -> GND
- D6 pad 1: /BYPASS-BTN -> BATT+PROT
- D8 pad 1: Net-(D8-K) -> Net-(D7-K)
- D8 pad 2: Net-(D7-A) -> Net-(D8-A)
- D9 pad 1: Net-(D9-K) -> Net-(D10-K)
- D9 pad 2: Net-(D10-A) -> Net-(D9-A)
- Q1 pad 1: Net-(Q1-G) -> Net-(D1-A)
- Q1 pad 2: Net-(D1-A) -> Net-(D1-K)
- Q1 pad 3: BATT+PROT -> BATT+
- Q10 pad 1: Net-(D19-K) -> Net-(D24-K)
- Q10 pad 3: /BYPASS-BTN -> Net-(D19-K)
- Q11 pad 1: Net-(D20-A) -> Net-(D25-K)
- Q11 pad 2: BATT+PROT -> GND
- Q11 pad 3: Net-(Q11-D) -> Net-(D21-K)
- Q12 pad 1: Net-(D21-A) -> Net-(D26-A)
- Q13 pad 1: Net-(D24-K) -> Net-(D29-K)
- Q13 pad 2: Net-(D24-A) -> GND
- Q13 pad 3: Net-(D22-K) -> Net-(D27-K)
- Q14 pad 1: Net-(D25-A) -> Net-(D30-A)
- Q15 pad 1: Net-(D28-K) -> Net-(D33-K)
- Q15 pad 2: Net-(D28-A) -> GND
- Q15 pad 3: Net-(D26-K) -> Net-(D31-K)
- Q16 pad 1: Net-(D29-A) -> Net-(D34-A)
- Q16 pad 3: Net-(D30-K) -> Net-(D35-K)
- Q17 pad 1: Net-(D30-A) -> Net-(D35-A)
- Q17 pad 2: Net-(D30-K) -> Net-(D35-K)
- Q18 pad 1: Net-(D31-A) -> Net-(D36-A)
- Q18 pad 2: /HVILS-A -> Net-(D36-K)
- Q18 pad 3: Net-(Q18-D) -> Net-(D50-K)
- Q19 pad 1: Net-(D32-A) -> Net-(D37-A)
- Q2 pad 1: Net-(Q2-G) -> Net-(D2-A)
- Q2 pad 2: Net-(D7-A) -> /IMD-Fault-Passthru/OUTPUT
- Q2 pad 3: BATT+PROT -> /HVILS-A
- Q20 pad 1: Net-(D33-A) -> Net-(D38-A)
- Q21 pad 1: Net-(D34-A) -> Net-(D39-A)
- Q22 pad 1: Net-(D45-A) -> Net-(D50-K)
- Q22 pad 2: BATT+PROT -> GND
- Q22 pad 3: /BMS-Fault-Passthru/INPUT -> Net-(D42-K)
- Q23 pad 1: Net-(D46-K) -> Net-(D51-A)
- Q23 pad 2: GND -> BATT+PROT
- Q23 pad 3: Net-(Q23-D) -> /BMS-Fault-Passthru/INPUT
- Q24 pad 1: Net-(D47-K) -> Net-(D52-K)
- Q24 pad 2: BATT+PROT -> GND
- Q24 pad 3: Net-(D47-A) -> Net-(Q24-D)
- Q3 pad 1: Net-(Q3-G) -> Net-(D3-K)
- Q3 pad 2: Net-(D10-A) -> GND
- Q3 pad 3: BATT+PROT -> /IMD-FAULT-VCU
- Q4 pad 1: Net-(D11-A) -> Net-(D4-K)
- Q4 pad 2: Net-(D11-K) -> GND
- Q4 pad 3: BATT+ -> /BYPASS-BTN
- Q5 pad 1: Net-(Q5-G) -> Net-(D5-K)
- Q5 pad 2: Net-(Q5-S) -> GND
- Q5 pad 3: BATT+PROT -> /BYPASS-BTN
- Q6 pad 1: Net-(Q6-G) -> Net-(D6-A)
- Q6 pad 2: Net-(Q6-S) -> BATT+PROT
- Q6 pad 3: BATT+PROT -> Net-(Q6-D)
- Q7 pad 1: Net-(D16-A) -> Net-(D15-K)
- Q7 pad 2: /IMD-Fault-Passthru/OUTPUT -> GND
- Q7 pad 3: /HVILS-A -> Net-(D7-K)
- Q8 pad 1: Net-(D17-K) -> Net-(D16-K)
- Q8 pad 3: /IMD-FAULT-VCU -> Net-(D10-K)
- Q9 pad 1: Net-(D18-K) -> Net-(D23-K)
- Q9 pad 3: /BYPASS-BTN -> Net-(D17-K)
- R1 pad 1: /PRECHARGE-DEBUG -> Net-(D1-K)
- R1 pad 2: Net-(Q1-G) -> BATT+PROT
- R10 pad 1: Net-(D5-A) -> Net-(Q6-D)
- R10 pad 2: BATT+PROT -> GND
- R11 pad 2: BATT+PROT -> Net-(C1-Pad2)
- R12 pad 1: GND -> Net-(C1-Pad2)
- R12 pad 2: Net-(D11-K) -> BATT+PROT
- R13 pad 1: Net-(D1-K) -> Net-(D7-A)
- R13 pad 2: GND -> BATT+PROT
- R14 pad 1: Net-(D2-K) -> Net-(D8-A)
- R14 pad 2: GND -> BATT+PROT
- R15 pad 1: Net-(D7-K) -> Net-(D9-A)
- R15 pad 2: GND -> BATT+PROT
- R16 pad 1: Net-(D8-K) -> Net-(D10-A)
- R16 pad 2: GND -> BATT+PROT
- R17 pad 1: Net-(D9-K) -> Net-(D11-A)
- R17 pad 2: GND -> BATT+
- R18 pad 1: Net-(D10-K) -> Net-(D12-A)
- R18 pad 2: GND -> BATT+
- R19 pad 1: GND -> Net-(D13-A)
- R19 pad 2: Net-(D11-A) -> BATT+PROT
- R2 pad 1: /POS-AIRS-DEBUG -> GND
- R2 pad 2: Net-(Q2-G) -> Net-(D1-K)
- R20 pad 1: /ACCY-FAN-ON -> Net-(D14-A)
- R20 pad 2: Net-(Q5-G) -> BATT+PROT
- R21 pad 1: /TRACTIVE-FAN-ON -> /ACCY-FAN-ON
- R21 pad 2: Net-(Q6-G) -> Net-(D15-K)
- R22 pad 1: GND -> /TRACTIVE-FAN-ON
- R22 pad 2: Net-(Q5-G) -> Net-(D16-K)
- R23 pad 2: Net-(Q6-G) -> Net-(D15-K)
- R24 pad 1: Net-(D12-A) -> GND
- R24 pad 2: Net-(Q5-S) -> Net-(D16-K)
- R25 pad 1: Net-(D13-A) -> Net-(D17-A)
- R25 pad 2: Net-(Q5-S) -> BATT+PROT
- R26 pad 1: Net-(D14-A) -> Net-(D18-A)
- R26 pad 2: Net-(Q6-S) -> BATT+PROT
- R27 pad 1: Net-(D15-A) -> Net-(D19-A)
- R27 pad 2: Net-(Q6-S) -> BATT+PROT
- R28 pad 1: Net-(D19-K) -> Net-(D20-A)
- R28 pad 2: /HVILS-A -> BATT+PROT
- R29 pad 1: /BYPASS-BTN -> Net-(D21-A)
- R3 pad 1: /NEG-AIRS-DEBUG -> GND
- R3 pad 2: Net-(Q3-G) -> Net-(D1-A)
- R30 pad 1: /BYPASS-BTN -> Net-(D22-A)
- R30 pad 2: Net-(D16-A) -> BATT+PROT
- R31 pad 1: Net-(D17-K) -> /PRECHARGE-DEBUG
- R31 pad 2: /IMD-FAULT -> Net-(D23-K)
- R32 pad 1: GND -> /NEG-AIRS-DEBUG
- R32 pad 2: /IMD-FAULT -> Net-(D24-K)
- R33 pad 1: Net-(Q11-D) -> /POS-AIRS-DEBUG
- R33 pad 2: Net-(D18-K) -> Net-(D25-K)
- R34 pad 1: Net-(Q11-D) -> GND
- R34 pad 2: GND -> Net-(D23-K)
- R35 pad 1: Net-(D20-A) -> GND
- R35 pad 2: Net-(C1-Pad2) -> Net-(D24-K)
- R36 pad 1: Net-(C1-Pad2) -> GND
- R36 pad 2: BATT+PROT -> Net-(D25-K)
- R37 pad 1: Net-(D22-A) -> GND
- R37 pad 2: BATT+PROT -> /BMS-Fault-Passthru/OUTPUT
- R38 pad 1: Net-(D23-A) -> Net-(D27-A)
- R39 pad 1: /BMS-FAULT -> Net-(D28-A)
- R4 pad 1: Net-(Q1-G) -> Net-(D5-K)
- R4 pad 2: GND -> /HVILS-A
- R40 pad 2: Net-(D21-A) -> Net-(D26-A)
- R41 pad 2: Net-(D24-K) -> BATT+PROT
- R42 pad 1: GND -> /BMS-FAULT
- R42 pad 2: Net-(D24-A) -> Net-(D29-K)
- R43 pad 1: Net-(D26-A) -> GND
- R43 pad 2: BATT+PROT -> /IMD-Fault-Passthru/OUTPUT
- R44 pad 1: Net-(D27-A) -> Net-(D31-A)
- R45 pad 1: /IMD-FAULT-VCU -> Net-(D32-A)
- R46 pad 2: Net-(D25-A) -> Net-(D30-A)
- R47 pad 2: Net-(D28-K) -> BATT+PROT
- R48 pad 1: GND -> /IMD-FAULT-VCU
- R48 pad 2: Net-(D28-A) -> Net-(D33-K)
- R49 pad 2: Net-(D29-A) -> Net-(D34-A)
- R5 pad 1: Net-(Q2-G) -> /BYPASS-BTN
- R5 pad 2: GND -> BATT+PROT
- R50 pad 2: Net-(D30-A) -> Net-(D35-A)
- R52 pad 1: Net-(D35-A) -> GND
- R52 pad 2: /SD-POWER -> /HVILS-A
- R53 pad 1: Net-(D36-A) -> Net-(D36-K)
- R53 pad 2: /SD-POWER -> /HVILS-A
- R54 pad 1: GND -> Net-(D40-A)
- R54 pad 2: /HVILS-A -> /SD-POWER
- R55 pad 1: /CRASH-SW-A -> Net-(D41-A)
- R55 pad 2: Net-(D31-A) -> /SD-POWER
- R56 pad 1: /BOTS-A -> /CRASH-SW-A
- R56 pad 2: Net-(D32-A) -> Net-(D36-A)
- R57 pad 1: /BOTS-B -> /BOTS-A
- R57 pad 2: Net-(D33-A) -> Net-(D37-A)
- R58 pad 1: /SD-POWER -> /BOTS-B
- R58 pad 2: Net-(D34-A) -> Net-(D38-A)
- R59 pad 1: GND -> /SD-POWER
- R59 pad 2: /CRASH-SW-A -> Net-(D39-A)
- R6 pad 1: Net-(Q3-G) -> /BYPASS-BTN
- R6 pad 2: GND -> Net-(D2-A)
- R60 pad 2: /BOTS-A -> Net-(D36-K)
- R61 pad 2: /BOTS-B -> /CRASH-SW-A
- R62 pad 2: /SD-POWER -> /BOTS-A
- R63 pad 1: Net-(D37-A) -> GND
- R63 pad 2: Net-(Q18-D) -> /BOTS-B
- R64 pad 1: Net-(D38-A) -> GND
- R64 pad 2: Net-(Q18-D) -> /SD-POWER
- R65 pad 1: Net-(D39-A) -> Net-(D42-A)
- R65 pad 2: Net-(Q19-D) -> /HVILS-A
- R66 pad 1: Net-(D40-A) -> Net-(D43-A)
- R66 pad 2: Net-(Q19-D) -> /HVILS-A
- R67 pad 1: Net-(D41-A) -> Net-(D44-A)
- R67 pad 2: Net-(Q20-D) -> Net-(Q19-D)
- R68 pad 1: Net-(D42-A) -> Net-(D45-A)
- R68 pad 2: Net-(Q20-D) -> Net-(Q19-D)
- R69 pad 1: Net-(D43-A) -> Net-(D46-A)
- R69 pad 2: Net-(Q21-D) -> Net-(Q20-D)
- R7 pad 1: Net-(D11-K) -> Net-(D3-K)
- R7 pad 2: BATT+PROT -> /IMD-FAULT
- R70 pad 1: Net-(D44-A) -> Net-(D47-A)
- R70 pad 2: Net-(Q21-D) -> Net-(Q20-D)
- R71 pad 1: Net-(Q23-D) -> Net-(D48-A)
- R71 pad 2: BATT+PROT -> Net-(Q21-D)
- R72 pad 1: Net-(Q23-D) -> Net-(D49-A)
- R72 pad 2: Net-(D45-A) -> Net-(Q21-D)
- R73 pad 1: /BSPD-FAULT-VCU -> GND
- R73 pad 2: Net-(D46-K) -> Net-(D50-K)
- R74 pad 2: /BSPD-FAULT-VCU -> /BMS-Fault-Passthru/INPUT
- R75 pad 1: /BSPD-FAULT-VCU -> Net-(Q24-D)
- R75 pad 2: Net-(D47-K) -> BATT+PROT
- R76 pad 1: Net-(D48-A) -> Net-(Q24-D)
- R76 pad 2: Net-(D47-A) -> Net-(D51-A)
- R77 pad 1: Net-(D49-A) -> /BSPD-FAULT-VCU
- R77 pad 2: Net-(D47-A) -> Net-(D52-K)
- R8 pad 1: Net-(D3-A) -> GND
- R8 pad 2: BATT+ -> /IMD-FAULT
- R9 pad 1: Net-(D4-A) -> Net-(Q6-D)
- R9 pad 2: BATT+ -> Net-(D4-K)
- VIN1 pad 1: Net-(D11-K) -> Net-(D1-K)
Routing:
- net (no net): track 0.00 -> 48.2 mm, vias 0 -> 2
- net /BMS-Fault-Passthru/OUTPUT: track 20.8 -> 30.9 mm, vias 0 -> 2
- net Net-(D30-K): track 10.1 -> 0.00 mm, vias 2 -> 0
- net Net-(D16-A): track 7.56 -> 0.00 mm
- net Net-(D29-A): track 6.98 -> 0.00 mm
- net /HVILS-A: track 86.6 -> 93.2 mm, vias 2 -> 4
- net Net-(D33-A): track 5.48 -> 0.00 mm
- net Net-(Q18-D): track 5.46 -> 0.00 mm, vias 1 -> 0
- net Net-(Q6-D): track 0.00 -> 5.29 mm, vias 0 -> 2
- net Net-(D25-A): track 4.50 -> 0.00 mm
- net Net-(D7-K): track 2.04 -> 6.12 mm
- net Net-(D8-K): track 4.08 -> 0.00 mm
- net Net-(D28-A): track 3.95 -> 0.00 mm
- net Net-(D24-A): track 3.95 -> 0.00 mm
- net Net-(Q6-G): track 3.86 -> 0.00 mm
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Other:
- board text added: "MK.11 Shutdown V2"
- board text removed: "MK.11 Shutdown V1"

Commit message: layout done extra crispy v2
Parts:
- D12, D14, D18, D20, D22, D28, D32, D41, D43, D45, D47, D55, R20, R26, R28, R30, R39, R45, R55, R72, R81: moved to B.Cu
- D13, D15, D2, D23, D27, D36, D38, D4, D40, D42, D44, D6, R11, R25, R27, R38, R44, R53, R64, R77, R9: moved to F.Cu
- R60: value 20k -> 13k
- moved D23 134.7 mm to (133.8, 171.1), turned to -90 degrees
- moved D24 126.2 mm to (146.5, 171.1), turned to -90 degrees
- moved D21 113.4 mm to (162.2, 175.5), turned to -90 degrees
- moved D17 108.0 mm to (137.2, 175.5)
- moved R31 107.3 mm to (136.9, 169.1)
- moved D22 107.0 mm to (162.2, 175.5), turned to -90 degrees
- moved D49 107.0 mm to (180.2, 155.8), turned to -90 degrees
- moved D48 106.9 mm to (180.3, 155.8), turned to -90 degrees
- moved R78 104.6 mm to (290.7, 176.3)
- moved R6 103.5 mm to (239.9, 170.1), turned to 90 degrees
- moved R71 102.7 mm to (182.4, 155.8)
- moved Q25 102.5 mm to (285.1, 175.0), turned to 90 degrees
- moved R34 101.9 mm to (136.9, 167.5), turned to 180 degrees
- moved R72 101.1 mm to (182.3, 155.8)
- moved D55 100.6 mm to (285.0, 155.8), turned to -90 degrees
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Routing:
- net (no net): track 48.2 -> 0.00 mm, vias 2 -> 0
- net Net-(D31-K): track 0.00 -> 38.4 mm, vias 1 -> 2
- net Net-(D27-K): track 0.00 -> 37.8 mm, vias 0 -> 2
- net /BOTS-A: track 88.1 -> 125.5 mm
- net /ACCY-FAN-ON: track 40.8 -> 72.1 mm, vias 0 -> 1
- net Net-(D42-K): track 0.00 -> 30.8 mm, vias 0 -> 2
- net Net-(D53-A): track 0.00 -> 28.7 mm, vias 0 -> 2
- net /TSSI-STATUS: track 120.3 -> 148.4 mm
- net /PRECHARGE-DEBUG: track 55.7 -> 83.4 mm, vias 1 -> 0
- net /BYPASS-BTN: track 130.8 -> 158.4 mm, vias 4 -> 2
- net /BOTS-B: track 98.8 -> 123.9 mm, vias 0 -> 1
- net /CRASH-SW-A: track 85.9 -> 110.8 mm
- net /BMS-FAULT: track 64.8 -> 86.1 mm, vias 3 -> 1
- net /NEG-AIRS-DEBUG: track 68.9 -> 52.7 mm, vias 2 -> 0
- net Net-(D35-K): track 0.00 -> 16.0 mm
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- added copper zone on F.Cu, net BATT+PROT
Other:
- board text added: "BMS1"
- board text added: "BOTS1"
- board text added: "BSPD1"
- board text added: "BYPASS1"
- board text added: "CS1"
- board text added: "HVILS1"
- board text added: "IMD1"
- board text added: "TSMS1"
