File: Shutdown-Circuit.kicad_sch (KiCad schematic)
At the start: 41 parts, among them Q20 SI2347DS-T1-GE3, Q21 SI2347DS-T1-GE3, Q22 SI2347DS-T1-GE3, Q23 SI2347DS-T1-GE3

Commit message: completed placement:
Parts:
- renumbered D34 to D32, D37 to D33, D40 to D34, D43 to D35, D44 to D36, D45 to D37, D32 to D38, D33 to D39, D35 to D40, D36 to D41, D38 to D42, D39 to D43, D41 to D44, D42 to D45, R93 to R76, R94 to R77, R76 to R78, R83 to R80, R87 to R81, R91 to R82, R80 to R83, R88 to R85, R92 to R86, R77 to R87, R78 to R88, R81 to R89, R82 to R90, R85 to R91, R86 to R92, R89 to R93, R90 to R94

Commit message: updated port directionalities, updated pinout
Changed lines of the file:
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@@
 	)
 	(hierarchical_label "SD-POWER"
-		(shape input)
+		(shape output)
 		(at 327.66 129.54 0)
 		(effects

Commit message: Schem is reannotated time to redo all of the layout
Parts:
- renumbered D32 to D26, D33 to D27, D34 to D28, D35 to D29, D36 to D30, D37 to D31, D38 to D32, D39 to D33, D40 to D34, D41 to D35, D42 to D36, D43 to D37, D44 to D38, D45 to D39, Q20 to Q18, Q21 to Q19, Q22 to Q20, Q23 to Q21, R76 to R47, R77 to R48, R78 to R49, R79 to R50, R80 to R51, R81 to R52, R82 to R53, R83 to R54, R84 to R55, R85 to R56, R86 to R57, R87 to R58, R88 to R59, R89 to R60, R90 to R61, R91 to R62, R92 to R63, R93 to R64, R94 to R65, TP24 to TP6, TP25 to TP7, TP26 to TP8, TP27 to TP9

Commit message: Finished shutdown, 0 drc, need to export gerbers
Parts:
- BOTS1: renamed from TP8; value ~ -> BOTS
- CS1: renamed from TP7; value ~ -> CS
- HVILS1: renamed from TP6; value ~ -> HVILS
- TSMS1: renamed from TP9; value ~ -> TSMS
- renumbered D26 to D31, D27 to D32, D28 to D33, D29 to D34, D30 to D35, D31 to D36, D32 to D37, D33 to D38, D34 to D39, D35 to D40, D36 to D41, D37 to D42, D38 to D43, D39 to D44, R47 to R52, R48 to R53, R49 to R54, R50 to R55, R51 to R56, R52 to R57, R53 to R58, R54 to R59, R55 to R60, R56 to R61, R57 to R62, R58 to R63, R59 to R64, R60 to R65, R61 to R66, R62 to R67, R63 to R68, R64 to R69, R65 to R70
Other:
- moved on the sheet: HVILS1

Commit message: schematic updated to V2 extra crispy
Parts:
- removed D35, D36, D37, D38, D39, D40, D41: Red, LED_SMD:LED_0805_2012Metric, symbol -Diodes-LED:NCD0805R1
- removed R52, R53, R63, R64, R65, R66, R67, R68, R69, R70: 510, Resistor_SMD:R_0603_1608Metric_Pad0.98x0.95mm_HandSolder, symbol -R-SMD-0603:R-0603-510-1%-100mW-100PPM
- removed R59: 1M, Resistor_SMD:R_0603_1608Metric_Pad0.98x0.95mm_HandSolder, symbol -R-SMD-0603:R-0603-1M-1%-100mW-100PPM
- removed R62: 100k, Resistor_SMD:R_0603_1608Metric_Pad0.98x0.95mm_HandSolder, symbol -R-SMD-0603:R-0603-100k-1%-100mW-100PPM
- added D40, D41: Green, LED_SMD:LED_0805_2012Metric, symbol -Diodes-LED:NCD0805G1
- added D45, D46, D47, D48, D49: Red, LED_SMD:LED_0805_2012Metric, symbol -Diodes-LED:NCD0805R1
- added D50: BZT52C16, Diode_SMD:D_SOD-123, symbol -Diodes-Zener:BZT52C16
- added Q22: SI2318CDS-T1-GE3, Package_TO_SOT_SMD:SOT-23-3, symbol -MOSFET-N-Channel:SI2318CDS-T1-GE3
- added R53, R64: 10k, Resistor_SMD:R_0603_1608Metric_Pad0.98x0.95mm_HandSolder, symbol -R-SMD-0603:R-0603-10k-1%-100mW-100PPM
- added R54, R55: 3.6k, Resistor_SMD:R_0603_1608Metric_Pad0.98x0.95mm_HandSolder, symbol -R-SMD-0603:R-0603-3.6k-1%-100mW-100PPM
- added R60: 20k, Resistor_SMD:R_0603_1608Metric_Pad0.98x0.95mm_HandSolder, symbol -R-SMD-0603:R-0603-20k-1%-100mW-100PPM
- added R61, R73: 100k, Resistor_SMD:R_0603_1608Metric_Pad0.98x0.95mm_HandSolder, symbol -R-SMD-0603:R-0603-100k-1%-100mW-100PPM
- added R65, R66, R67, R68, R69, R70, R71, R72: 680, Resistor_SMD:R_0603_1608Metric_Pad0.98x0.95mm_HandSolder, symbol -R-SMD-0603:R-0603-680-1%-100mW-100PPM
- D42, D43, D44: Digikey P/N 350-2039-1-ND -> 160-1427-1-ND; Mouser P/N 645-598-8120-107F -> 859-LTST-C171KRKT
- renumbered D31 to D36, D32 to D37, D33 to D38, D34 to D39, R54 to R52, R55 to R56, R56 to R57, R57 to R58, R58 to R59, R60 to R62, R61 to R63
Connections:
- net CS-A: now also R61.2
- net GND: now also D40.1 (K), D41.1 (K), D45.1 (K), D46.1 (K), D47.1 (K), D48.1 (K), D49.1 (K), D50.2 (A), Q22.2 (S), R60.1, R61.1, R64.1, R73.1; no longer D42.1 (K), D43.1 (K)
- net HVILS-A: now also R53.2, R65.2, R66.2; no longer D36.1 (K), Q18.2 (S)
- net SD-POWER: now also R54.2, R55.2, R64.2
- net at D43.2 (A): now also R66.1
- net at Q20.3 (D): now also R69.2, R70.2
- net at Q18.3 (D): now also D50.1 (K), Q22.1 (G), R73.2
- net at D42.2 (A): now also R65.1
- net at Q19.3 (D): now also R67.2, R68.2
- net at D44.2 (A): now also R67.1
- net at Q21.3 (D): now also R71.2, R72.2
- new net: D36.1 (K), Q18.2 (S), R53.1, R60.2
- new net: D41.2 (A), R55.1
- new net: D45.2 (A), R68.1
- new net: D42.1 (K), D43.1 (K), Q22.3 (D)
- new net: D46.2 (A), R69.1
- new net: D49.2 (A), R72.1
- new net: D40.2 (A), R54.1
- new net: D47.2 (A), R70.1
- new net: D48.2 (A), R71.1
Other:
- moved on the sheet: BOTS1, CS1, D36, D37, D38, D39, HVILS1, Q18, Q19, Q20, Q21, R52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

Commit message: layout done extra crispy v2
Parts:
- removed R60: 20k, Resistor_SMD:R_0603_1608Metric_Pad0.98x0.95mm_HandSolder, symbol -R-SMD-0603:R-0603-20k-1%-100mW-100PPM
- added R60: 13k, Resistor_SMD:R_0603_1608Metric_Pad0.98x0.95mm_HandSolder, symbol -R-SMD-0603:R-0603-13k-1%-100mW-100PPM
Connections:
- net GND: now also R60.1
- net at D36.1 (K), Q18.2 (S), R53.1: now also R60.2
Other:
- moved on the sheet: R63
