File: Shutdown.kicad_sch (KiCad schematic)
At the start: 36 parts, among them J1 0194270049, J2 0194270049, Q1 SI2347DS-T1-GE3, Q2 SI2347DS-T1-GE3, Q3 SI2318CDS-T1-GE3, Q4 SI2318CDS-T1-GE3, Q5 SI2318CDS-T1-GE3, Q6 SI2347DS-T1-GE3

Commit message: layout done extra crispy v2
Parts:
- R1: now fitted
Other:
- sheet TSSI-Status-Signal ports: added BMS-FAULT; removed BMS-FAULT-VCU
Changed lines of the file:
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@@
 	(text_box "NOTE: P-MOSFET w/ gate pulled up to Vcc (Vsource) is NO. Drive gate low to close. Zener protects against excessive Vgs."
 		(exclude_from_sim no)
-		(at 242.57 114.3 0)
+		(at 243.84 114.3 0)
 		(size 30.48 7.62)
 		(margins 0.9525 0.9525 0.9525 0.9525)
@@
 		(on_board yes)
 		(in_pos_files yes)
-		(dnp yes)
+		(dnp no)
 		(property "Reference" "R1"
 			(at 72.4448 52.0334 0)
@@
 			)
 		)
-		(pin "BMS-FAULT-VCU" input
-			(at 125.73 60.96 180)
+		(pin "TSSI-STATUS" output
+			(at 148.59 57.15 0)
 			(effects
 				(font
 					(size 1.27 1.27)
 				)
-				(justify left)
+				(justify right)
 			)
 		)
-		(pin "TSSI-STATUS" output
-			(at 148.59 57.15 0)
+		(pin "BMS-FAULT" input
+			(at 125.73 60.96 180)
 			(effects
 				(font
 					(size 1.27 1.27)
 				)
-				(justify right)
+				(justify left)
 			)
 		)
