File: TSSI-Status-Signal.kicad_sch (KiCad schematic)
At the start: 7 parts, among them Q16 SI2347DS-T1-GE3, Q17 SI2347DS-T1-GE3

Commit message: layout done extra crispy v2
Connections:
- net BMS-FAULT-VCU renamed BMS-FAULT
Changed lines of the file:
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@@
 		)
 	)
-	(hierarchical_label "BMS-FAULT-VCU"
+	(hierarchical_label "BMS-FAULT"
 		(shape input)
 		(at 186.69 160.02 180)
